File: _autosave-speeduino_ntv650.kicad_pcb (KiCad board)
At the start: 2 copper layers, 74 x 119 mm, 78 parts, among them IC1 SP721, IC2 TC4424, J1 DB25_Female_MountingHoles, J2 Conn_01x01, J3 Conn_01x01, J4 Conn_01x01, J5 Conn_01x01, J6 Conn_01x01, J7 Conn_01x01, P1 MAX9926_9927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

Commit message: new element positions for 0.6 mm lines on pcb
Other:
- net class Default: trace_width 0.55 -> 0.6
Changed lines of the file:
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@@
   (net_class Default "Это класс цепей по умолчанию."
     (clearance 0.2)
-    (trace_width 0.55)
+    (trace_width 0.6)
     (via_dia 1.2)
     (via_drill 0.2)
